File: MCU.kicad_sch (KiCad schematic)
At the start: 81 parts, among them J402 RS485_1, J403 RS485_2, J404 Conn_ARM_JTAG_SWD_10, U403 EFM32PG22C200F512IM40, U404 SN75176AD, U405 XC6204B33, Y401 Abracon_ABM11

Commit message: Fixes.
Parts:
- removed TP?: TestPoint_Small, symbol 4ms_Connector:TestPoint_Small
- added F?: TODO, Fuse:Fuse_2920_7451Metric_Pad2.10x5.45mm_HandSolder, symbol Device:Polyfuse_Small
- added TP?: TestPoint_Small, symbol 4ms_Connector:TestPoint_Small
Connections:
- net +5V: now also F?.1; no longer J?.1 (Pin_1)
- net VCC_AUX: no longer C?.1, R?.1, R?.1, R?.1, R?.1, R?.1, R?.1, R?.1, U?.21 (VCC)
- net VCC_MCU: now also C?.1, R?.1, R?.1, R?.1, R?.1, R?.1, R?.1, R?.1, U?.21 (VCC)
- net at U403.40 (PD00): now also TP?.1
- new net: F?.2, J?.1 (Pin_1)
Other:
- title: Generator 0.0125 - 6.4 GHz (0.02 - 9.8 GHz) -> Generator 0.0125 - 6.4 GHz (or up to 20 GHz)
- moved on the sheet: C405, D411A, D411B, D411C, D411D, J402, J403, R416, R417, R418, U404
