File: input_clocks.kicad_sch (KiCad schematic)
At the start: 90 parts, among them J201 REFIN, J202 REFIN_DIRECT_P, J203 REFIN_DIRECT_N, J208 VTUNE, Q501 BFP181, Q502 BFP181, T201 TC2-1T+, U203 TSV914, U204 74LVC1G66, U501 LT1461AxS8-3.3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

Commit message: Schematic ready for impoting changes into PCB.
Parts:
- X201: symbol petr_lib_nightly:XTCLH40M000CHJA0P0 -> petr:XTCLH40M000CHJA0P0
Changed lines of the file:
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@@
     (rev "211230-001")
     (company "Petr Polasek")
-    (comment 1 "001, 2021-12-30 00:50")
+    (comment 1 "001, 2021-12-30 01:03")
     (comment 2 "TCXO / external input")
     (comment 3 "LMX2572 (6.4 GHz) / LMX2592 (9.8GHz) / LMX2594 (15 GHz) / LMX2595 (20 GHz)")
@@
     (pin "2")
   )
-  (symbol (lib_id "petr_lib_nightly:XTCLH40M000CHJA0P0") (at 229.87 99.06 0) (unit 1)
+  (symbol (lib_id "petr:XTCLH40M000CHJA0P0") (at 229.87 99.06 0) (unit 1)
     (in_bom yes) (on_board yes)
     (property "Reference" "X201" (id 0) (at 231.14 105.41 0)

Commit message: Synchronised PCB and schematic.
Parts:
- removed D201: 1.5KE51CA, Diode_THT:D_DO-201AE_P15.24mm_Horizontal, symbol Diode:1.5KExxCA
- added D503: SMAJ48CA, Diode_SMD_AKL:D_SMA_TVS, symbol Diode_TVS_AKL:SMAJ48CA
- J201: footprint petr_kicad:SMA_rosenberger_hybrid -> petr:SMA_rosenberger_hybrid
Connections:
- net GND: now also D503.2 (A)
- net REFIN_GND: now also D503.1 (K)
Changed lines of the file:
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@@
-    (pin "2")
-  )
-  (symbol (lib_id "Diode:1.5KExxCA") (at 30.48 166.37 270) (unit 1)
-    (in_bom yes) (on_board yes)
-    (property "Reference" "D201" (id 0) (at 32.4866 165.2016 90)
-      (effects (font (size 1.27 1.27)) (justify left))
-    )
-    (property "Value" "1.5KE51CA" (id 1) (at 32.4866 167.513 90)
-      (effects (font (size 1.27 1.27)) (justify left))
-    )
-    (property "Footprint" "Diode_THT:D_DO-201AE_P15.24mm_Horizontal" (id 2) (at 25.4 166.37 0)
-      (effects (font (size 1.27 1.27)) hide)
-    )
-    (property "Datasheet" "https://www.vishay.com/docs/88301/15ke.pdf" (id 3) (at 30.48 166.37 0)
-      (effects (font (size 1.27 1.27)) hide)
-    )
-    (pin "1")
     (pin "2")
   )
@@
     (property "Reference" "J201" (id 0) (at 20.8788 146.3548 0))
     (property "Value" "REFIN" (id 1) (at 20.8788 148.6662 0))
-    (property "Footprint" "petr_kicad:SMA_rosenberger_hybrid" (id 2) (at 16.51 143.51 0)
+    (property "Footprint" "petr:SMA_rosenberger_hybrid" (id 2) (at 16.51 143.51 0)
       (effects (font (size 1.27 1.27)) hide)
     )
@@
       (effects (font (size 1.27 1.27)) hide)
     )
+    (pin "1")
+    (pin "2")
+  )
+  (symbol (lib_id "Diode_TVS_AKL:SMAJ48CA") (at 30.48 166.37 270) (unit 1)
+    (in_bom yes) (on_board yes) (fields_autoplaced)
+    (property "Reference" "D503" (id 0) (at 33.02 165.0999 90)
+      (effects (font (size 1.27 1.27)) (justify left))
+    )
+    (property "Value" "SMAJ48CA" (id 1) (at 33.02 167.6399 90)
+      (effects (font (size 1.27 1.27)) (justify left))
+    )
+    (property "Footprint" "Diode_SMD_AKL:D_SMA_TVS" (id 2) (at 30.48 166.37 0)
+      (effects (font (size 1.27 1.27)) hide)
+    )
+    (property "Datasheet" "https://www.tme.eu/Document/dbc72d81c249fe51b6ab42300e8e06d0/SMAJ_ser.pdf" (id 3) (at 30.48 166.37 0)
+      (effects (font (size 1.27 1.27)) hide)
+    )
