File: MWGEN-G1.kicad_pcb (KiCad board)
At the start: 4 copper layers, 295 parts, among them J101 Conn_02x25_Odd_Even, J201 REFIN, J202 REFIN_DIRECT_P, J203 REFIN_DIRECT_N, J204 REFOUT_AUX_P, J205 REFOUT_AUX_N, J206 RFShield_TwoPieces, J207 REFOUT, J208 VTUNE, J209 DNP, J301 Vtune, J302 RFShield_TwoPieces, J303 CPout, J304 DNP, J305 DNP, J306 DNP, J307 DNP, J308 DNP, Q101 BSS138, Q102 BSS138, T201 TC2-1T+, T202 TC2-1T+, U201 Si53301, U202 XC6204B33, U203 TSV914, U204 74LVC1G66, U301 LMX2572, U302 XC6204B33, X201 XTCLH40M000CHJA0P0

Commit message: Schematic fixes
Parts:
- removed R217, R218: DNP, Resistor_SMD:R_0603_1608Metric_Pad0.98x0.95mm_HandSolder
- added C336: 10n, Capacitor_SMD:C_0603_1608Metric_Pad1.08x0.95mm_HandSolder, F.Cu at (200.4, 106.8)
- added C337: 10n, Capacitor_SMD:C_0603_1608Metric_Pad1.08x0.95mm_HandSolder, F.Cu at (200.8, 92.5)
- added C339: 10n, Capacitor_SMD:C_0603_1608Metric_Pad1.08x0.95mm_HandSolder, F.Cu at (200.8, 99.4)
- added J309: RFShield_TwoPieces, RF_Shielding:Laird_Technologies_BMI-S-205-F_38.10x25.40mm, B.Cu at (196.1, 98.0)
- C201, C202, C204, C207, C209, C212, C215, C311, C312, C314, C316, C317, C319, C320, C321, C323, C327, C328, C329, C330, C331, C332, C333, C334, C335, FB201, FB202, FB203, FB301, FB302, FB303, FB304, FB305, FB306, R205, R206, R209, R320, R326, R328, R329, R331, R332: moved to B.Cu
- J202, J203: footprint petr_kicad:SMA_rosenberger_hybrid -> Connector_Coaxial:U.FL_Molex_MCRF_73412-0110_Vertical
- J206, J302: footprint RF_Shielding:Laird_Technologies_BMI-S-206-F_36.83x33.68mm -> RF_Shielding:Laird_Technologies_BMI-S-205-F_38.10x25.40mm
- moved U204 157.1 mm to (229.6, 41.3)
- moved D101 145.6 mm to (216.2, -53.5)
- moved D102 145.6 mm to (217.3, -60.5)
- moved D103 145.6 mm to (242.3, -62.5)
- moved D106 145.6 mm to (250.4, -62.5)
- moved F101 145.6 mm to (217.2, -73.0)
- moved FB101 145.6 mm to (213.6, -65.3)
- moved Q101 145.6 mm to (241.9, -67.8)
- moved Q102 145.6 mm to (250.4, -67.8)
- moved R101 145.6 mm to (242.4, -73.5)
- moved R102 145.6 mm to (242.2, -58.8)
- moved R104 145.6 mm to (250.4, -73.5)
- moved R106 145.6 mm to (250.2, -58.5)
- moved R124 145.6 mm to (230.7, -74.5)
- moved R131 145.6 mm to (230.2, -69.0)
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Connections:
- R220 pad 2: Net-(R217-Pad1) -> /Clock reference/CLKIN_1
- R221 pad 1: Net-(R218-Pad1) -> /Clock reference/~CLKIN_1
- R222 pad 1: Net-(R217-Pad1) -> /Clock reference/CLKIN_1
- R223 pad 1: Net-(R218-Pad1) -> /Clock reference/~CLKIN_1
- R253 pad 1: /VCC_fREF -> /Clock reference/VDD_TCXO
- R255 pad 1: /VCC_fREF -> /Clock reference/VDD_TCXO
Routing:
- net /PLL/VCC_PLL: track 0.00 -> 49.9 mm, vias 0 -> 3
- net /PLL/VccBUF: track 0.00 -> 41.2 mm, vias 0 -> 4
- net /PLL/Vtune: track 0.00 -> 24.6 mm, vias 0 -> 2
- net /PLL/~RFoutA: track 0.00 -> 24.3 mm
- net /PLL/RFoutB: track 0.00 -> 24.3 mm
- net /PLL/~RFoutB: track 0.00 -> 24.2 mm
- net /PLL/RFoutA: track 0.00 -> 24.2 mm
- net Net-(C306-Pad2): track 0.00 -> 17.7 mm
- net Net-(C307-Pad2): track 0.00 -> 17.7 mm
- net /PLL/MUXout: track 0.00 -> 15.9 mm, vias 0 -> 2
- net Net-(C308-Pad2): track 0.00 -> 15.5 mm
- net Net-(C309-Pad2): track 0.00 -> 15.0 mm
- net /PLL/CSB: track 0.00 -> 14.2 mm, vias 0 -> 2
- net GND: track 0.00 -> 14.1 mm, vias 0 -> 231
- net /PLL/SDI: track 0.00 -> 12.9 mm
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- added copper zone on B.Cu, net GND
- added copper zone on F.Cu, net GND
- added copper zone on In1.Cu, net GND
- added copper zone on In2.Cu, net GND
Other:
- board outline added: 100 x 100 mm
- board text added: "CHA_N"
- board text added: "CHA_P"
- board text added: "CHB_N"
- board text added: "CHB_P"
- board text added: "CPout"
- board text added: "Vtune"

Commit message: Schematic checked. All footprints assigned. Electrolytics need footprint check, so do the RS485 and power connectors and the MuRata oscillator (also it is now EOL) and the crystal. The power protection transils on aux input/output need replacement. PCB in sync with SCH.
Parts:
- added C401: 100n, Capacitor_SMD:C_0603_1608Metric_Pad1.08x0.95mm_HandSolder, F.Cu at (368.3, 101.6)
- added C402: 100n, Capacitor_SMD:C_0603_1608Metric_Pad1.08x0.95mm_HandSolder, F.Cu at (366.2, 91.6)
- added C403: 100n, Capacitor_SMD:C_0603_1608Metric_Pad1.08x0.95mm_HandSolder, F.Cu at (359.6, 104.8)
- added C404: 100n, Capacitor_SMD:C_0603_1608Metric_Pad1.08x0.95mm_HandSolder, F.Cu at (348.8, 112.2)
- added C405: 100n, Capacitor_SMD:C_0603_1608Metric_Pad1.08x0.95mm_HandSolder, F.Cu at (376.5, 81.8)
- added C406: 100u, Capacitor_SMD:CP_Elec_6.3x7.7, F.Cu at (348.3, 94.0)
- added C407: 10u, Capacitor_SMD:C_0805_2012Metric_Pad1.18x1.45mm_HandSolder, F.Cu at (335.7, 91.4)
- added C408: 100n, Capacitor_SMD:C_0603_1608Metric_Pad1.08x0.95mm_HandSolder, F.Cu at (375.3, 87.6)
- added C409: 100n, Capacitor_SMD:C_0603_1608Metric_Pad1.08x0.95mm_HandSolder, F.Cu at (389.5, 79.2)
- added C410: 100n, Capacitor_SMD:C_0603_1608Metric_Pad1.08x0.95mm_HandSolder, F.Cu at (358.3, 109.9)
- added C411: 100n, Capacitor_SMD:C_0603_1608Metric_Pad1.08x0.95mm_HandSolder, F.Cu at (357.5, 112.4)
- added C412: 1n, Capacitor_SMD:C_0603_1608Metric_Pad1.08x0.95mm_HandSolder, F.Cu at (354.0, 107.4)
- added C413: 4u7, Capacitor_SMD:C_0603_1608Metric_Pad1.08x0.95mm_HandSolder, F.Cu at (358.4, 107.4)
- added C414: 4u7, Capacitor_SMD:C_0603_1608Metric_Pad1.08x0.95mm_HandSolder, F.Cu at (373.2, 96.6)
- added C415: 2u2, Capacitor_SMD:C_0805_2012Metric_Pad1.18x1.45mm_HandSolder, F.Cu at (340.5, 91.4)
- added C416: 2u2, Capacitor_SMD:C_0805_2012Metric_Pad1.18x1.45mm_HandSolder, F.Cu at (330.9, 91.4)
- added C417: 100n, Capacitor_SMD:C_0603_1608Metric_Pad1.08x0.95mm_HandSolder, F.Cu at (368.8, 99.1)
- added C418: 10u, Capacitor_SMD:C_0805_2012Metric_Pad1.18x1.45mm_HandSolder, F.Cu at (350.2, 88.4)
- added C419: 100u, Capacitor_SMD:CP_Elec_6.3x7.7, F.Cu at (358.8, 90.9)
- added C501: 100n, Capacitor_SMD:C_0603_1608Metric_Pad1.08x0.95mm_HandSolder, F.Cu at (338.1, 126.8)
- added C502: 1n, Capacitor_SMD:C_0603_1608Metric_Pad1.08x0.95mm_HandSolder, F.Cu at (340.4, 129.3)
- added C503: 100n, Capacitor_SMD:C_0603_1608Metric_Pad1.08x0.95mm_HandSolder, F.Cu at (330.4, 135.8)
- added C504: 100n, Capacitor_SMD:C_0603_1608Metric_Pad1.08x0.95mm_HandSolder, F.Cu at (345.8, 119.7)
- added D401: , LED_SMD:LED_0603_1608Metric_Pad1.05x0.95mm_HandSolder, F.Cu at (340.1, 113.7)
- added D402: , LED_SMD:LED_0603_1608Metric_Pad1.05x0.95mm_HandSolder, F.Cu at (335.7, 111.1)
- added D403: , LED_SMD:LED_0603_1608Metric_Pad1.05x0.95mm_HandSolder, F.Cu at (340.1, 111.1)
- added D404: , LED_SMD:LED_0603_1608Metric_Pad1.05x0.95mm_HandSolder, F.Cu at (345.3, 107.2)
- added D405: , LED_SMD:LED_0603_1608Metric_Pad1.05x0.95mm_HandSolder, F.Cu at (331.3, 111.1)
- added D406: , LED_SMD:LED_0603_1608Metric_Pad1.05x0.95mm_HandSolder, F.Cu at (376.5, 76.7)
- added D407: , LED_SMD:LED_0603_1608Metric_Pad1.05x0.95mm_HandSolder, F.Cu at (331.3, 113.7)
- added D408: , LED_SMD:LED_0603_1608Metric_Pad1.05x0.95mm_HandSolder, F.Cu at (355.3, 102.3)
- added D409: PESD3V3L4UG, Package_TO_SOT_SMD:SOT-353_SC-70-5, F.Cu at (383.9, 87.5)
- added D411: PESD3V3L4UG, Package_TO_SOT_SMD:SOT-353_SC-70-5, F.Cu at (362.7, 108.0)
- added D412: PESD3V3L4UG, Package_TO_SOT_SMD:SOT-353_SC-70-5, F.Cu at (379.6, 90.0)
- added D413: MCU_ON, LED_SMD:LED_0603_1608Metric_Pad1.05x0.95mm_HandSolder, F.Cu at (335.7, 113.7)
- added D501: BAT54S, Package_TO_SOT_SMD:SOT-23, F.Cu at (341.2, 120.7)
- added D502: TCXO_ON, LED_SMD:LED_0603_1608Metric_Pad1.05x0.95mm_HandSolder, F.Cu at (326.0, 134.3)
- added FB401: TODO, Inductor_SMD:L_0603_1608Metric_Pad1.05x0.95mm_HandSolder, F.Cu at (354.0, 109.9)
- added FB501: TODO, Inductor_SMD:L_0603_1608Metric_Pad1.05x0.95mm_HandSolder, F.Cu at (331.6, 130.7)
- added J401: Conn_01x07, Connector_PinHeader_2.54mm:PinHeader_1x07_P2.54mm_Vertical, F.Cu at (326.1, 77.7)
- added J402: Conn_01x03, Connector_Phoenix_MSTB:PhoenixContact_MSTBA_2,5_3-G-5,08_1x03_P5.08mm_Horizontal, F.Cu at (328.4, 98.8)
- added J403: Conn_01x03, Connector_Phoenix_MSTB:PhoenixContact_MSTBA_2,5_3-G-5,08_1x03_P5.08mm_Horizontal, F.Cu at (333.0, 78.9)
- added J404: Conn_ARM_JTAG_SWD_10, Connector_PinHeader_1.27mm:PinHeader_2x05_P1.27mm_Vertical_SMD, F.Cu at (369.5, 79.6)
- added JP501: SolderJumper_3_Bridged12, Jumper:SolderJumper-3_P1.3mm_Bridged12_RoundedPad1.0x1.5mm_NumberLabels, F.Cu at (333.1, 126.7)
- added JP502: SolderJumper_3_Bridged12, Jumper:SolderJumper-3_P1.3mm_Bridged12_RoundedPad1.0x1.5mm_NumberLabels, F.Cu at (326.6, 131.3)
- added JP503: SolderJumper_2_Bridged, Jumper:SolderJumper-2_P1.3mm_Bridged_RoundedPad1.0x1.5mm, F.Cu at (340.4, 134.8)
- added L401: 2u2, Inductor_SMD:L_1008_2520Metric_Pad1.43x2.20mm_HandSolder, F.Cu at (326.5, 111.7)
- added Q501: BFP181, Package_TO_SOT_SMD:SOT-23_Handsoldering, F.Cu at (327.1, 127.2)
- added Q502: BFP181, Package_TO_SOT_SMD:SOT-23_Handsoldering, F.Cu at (335.5, 120.8)
- added R217: DNP, Resistor_SMD:R_0603_1608Metric_Pad0.98x0.95mm_HandSolder, F.Cu at (344.7, 129.2)
- added R218: DNP, Resistor_SMD:R_0603_1608Metric_Pad0.98x0.95mm_HandSolder, F.Cu at (338.1, 124.3)
- added R401: 100, Resistor_SMD:R_0603_1608Metric_Pad0.98x0.95mm_HandSolder, F.Cu at (389.6, 76.7)
- added R402: 100, Resistor_SMD:R_0603_1608Metric_Pad0.98x0.95mm_HandSolder, F.Cu at (380.8, 79.2)
- added R403: 100, Resistor_SMD:R_0603_1608Metric_Pad0.98x0.95mm_HandSolder, F.Cu at (385.2, 79.2)
- added R404: 10k, Resistor_SMD:R_0603_1608Metric_Pad0.98x0.95mm_HandSolder, F.Cu at (385.2, 76.7)
- added R405: 3k3, Resistor_SMD:R_0603_1608Metric_Pad0.98x0.95mm_HandSolder, F.Cu at (379.6, 86.8)
- added R406: 2k, Resistor_SMD:R_0603_1608Metric_Pad0.98x0.95mm_HandSolder, F.Cu at (344.5, 112.2)
- added R407: 2k, Resistor_SMD:R_0603_1608Metric_Pad0.98x0.95mm_HandSolder, F.Cu at (373.2, 94.1)
- added R408: 2k, Resistor_SMD:R_0603_1608Metric_Pad0.98x0.95mm_HandSolder, F.Cu at (385.2, 81.7)
- added R409: 2k, Resistor_SMD:R_0603_1608Metric_Pad0.98x0.95mm_HandSolder, F.Cu at (363.9, 104.8)
- added R410: 2k, Resistor_SMD:R_0603_1608Metric_Pad0.98x0.95mm_HandSolder, F.Cu at (349.7, 107.1)
- added R411: 2k, Resistor_SMD:R_0603_1608Metric_Pad0.98x0.95mm_HandSolder, F.Cu at (376.5, 79.2)
- added R412: 2k, Resistor_SMD:R_0603_1608Metric_Pad0.98x0.95mm_HandSolder, F.Cu at (384.0, 84.3)
- added R413: 2k, Resistor_SMD:R_0603_1608Metric_Pad0.98x0.95mm_HandSolder, F.Cu at (375.3, 90.1)
- added R414: 10k, Resistor_SMD:R_0603_1608Metric_Pad0.98x0.95mm_HandSolder, F.Cu at (368.8, 96.6)
- added R415: 100, Resistor_SMD:R_0603_1608Metric_Pad0.98x0.95mm_HandSolder, F.Cu at (364.5, 96.3)
- added R416: 10k, Resistor_SMD:R_0603_1608Metric_Pad0.98x0.95mm_HandSolder, F.Cu at (353.2, 112.4)
- added R417: 10k, Resistor_SMD:R_0603_1608Metric_Pad0.98x0.95mm_HandSolder, F.Cu at (380.8, 81.8)
- added R418: 10k, Resistor_SMD:R_0603_1608Metric_Pad0.98x0.95mm_HandSolder, F.Cu at (359.6, 102.3)
- added R419: NC, Resistor_SMD:R_0603_1608Metric_Pad0.98x0.95mm_HandSolder, F.Cu at (364.5, 98.8)
- added R420: 1k, Resistor_SMD:R_0603_1608Metric_Pad0.98x0.95mm_HandSolder, F.Cu at (368.8, 94.1)
- added R421: 100, Resistor_SMD:R_0603_1608Metric_Pad0.98x0.95mm_HandSolder, F.Cu at (349.6, 109.7)
- added R422: 100, Resistor_SMD:R_0603_1608Metric_Pad0.98x0.95mm_HandSolder, F.Cu at (355.2, 104.9)
- added R423: 100, Resistor_SMD:R_0603_1608Metric_Pad0.98x0.95mm_HandSolder, F.Cu at (345.3, 109.7)
- added R424: 100, Resistor_SMD:R_0603_1608Metric_Pad0.98x0.95mm_HandSolder, F.Cu at (363.9, 102.3)
- added R425: 0R, Resistor_SMD:R_0603_1608Metric_Pad0.98x0.95mm_HandSolder, F.Cu at (379.6, 84.3)
- added R426: 2k, Resistor_SMD:R_0603_1608Metric_Pad0.98x0.95mm_HandSolder, F.Cu at (370.5, 91.6)
- added R427: 100, Resistor_SMD:R_0603_1608Metric_Pad0.98x0.95mm_HandSolder, F.Cu at (380.9, 76.7)
- added R428: 10k, Resistor_SMD:R_0603_1608Metric_Pad0.98x0.95mm_HandSolder, F.Cu at (375.3, 85.1)
- added R501: 33R, Resistor_SMD:R_0603_1608Metric_Pad0.98x0.95mm_HandSolder, F.Cu at (342.4, 124.2)
- added R502: 10k, Resistor_SMD:R_0603_1608Metric_Pad0.98x0.95mm_HandSolder, F.Cu at (331.6, 133.2)
- added R503: 1k, Resistor_SMD:R_0603_1608Metric_Pad0.98x0.95mm_HandSolder, F.Cu at (336.0, 129.7)
- added R504: TODO, Resistor_SMD:R_0603_1608Metric_Pad0.98x0.95mm_HandSolder, F.Cu at (334.7, 135.8)
- added R505: 2k, Resistor_SMD:R_0603_1608Metric_Pad0.98x0.95mm_HandSolder, F.Cu at (340.4, 131.8)
- added R506: DNP, Resistor_SMD:R_0603_1608Metric_Pad0.98x0.95mm_HandSolder, F.Cu at (342.4, 126.7)
- added R507: DNP, Resistor_SMD:R_0603_1608Metric_Pad0.98x0.95mm_HandSolder, F.Cu at (336.0, 132.2)
- added U401: 74HC4094, Package_SO:SO-16_3.9x9.9mm_P1.27mm, F.Cu at (352.0, 81.1)
- added U402: 74HC4094, Package_SO:SO-16_3.9x9.9mm_P1.27mm, F.Cu at (360.4, 81.1)
- added U403: efm32pg22c200f512im40-c, EFM32PG22C200:efm32pg22c200f512im40-c, F.Cu at (349.1, 102.0)
- added U404: SN75176AD, Package_SO:SOIC-8_3.9x4.9mm_P1.27mm, F.Cu at (368.9, 87.1)
- added U405: XC6204B33, Package_TO_SOT_SMD:SOT-89-5_Handsoldering, F.Cu at (357.9, 98.0)
- added U501: LT1461AxS8-3.3, Package_SO:SOIC-8_3.9x4.9mm_P1.27mm, F.Cu at (328.1, 121.7)
- added Y401: 38.4 MHz, Crystal:Crystal_SMD_2016-4Pin_2.0x1.6mm, F.Cu at (389.3, 82.2)
- C101: value TODO -> 100n
- C122, C123: value TODO -> 1n
- C231: footprint Capacitor_SMD:C_0603_1608Metric_Pad1.08x0.95mm_HandSolder -> Capacitor_SMD:C_0805_2012Metric_Pad1.18x1.45mm_HandSolder
- D202, D203: value BAV99 -> BAT54S
- J101: value Conn_02x25_Odd_Even -> Conn_01x02; footprint Connector_Multicomp:Multicomp_MC9A12-5034_2x25_P2.54mm_Vertical -> Connector_Phoenix_MSTB:PhoenixContact_MSTBA_2,5_2-G-5,08_1x02_P5.08mm_Horizontal
- J208: footprint petr_kicad:SMA_rosenberger_hybrid -> Connector_Coaxial:U.FL_Molex_MCRF_73412-0110_Vertical
- R102, R106: value 3k3 -> 2k
- R103, R105: value TODO -> 10k
- R107, R109, R110: value TODO -> 3k
- R108: value TODO -> 300
- R128: value DNP -> 0R
- R131, R132: value 3k3 -> 300
- R203: value 3R -> DNP
- R208: value DNP -> 56R
Connections:
- net /Clock reference/DUTY_ERROR renamed /Clock reference/Input Clocks/DUTY_ERROR
- net /Clock reference/TCXO_OUT renamed /Clock reference/Input Clocks/TCXO_OUT
- net /Clock reference/VCC/2 renamed /Clock reference/Input Clocks/VCC/2
- net /Clock reference/~CLKIN_0 renamed /Clock reference/~{CLKIN_0}
- net /PLL/~RFoutA renamed /PLL/~{RFoutA}
- net /PLL/~RFoutB renamed /PLL/~{RFoutB}
- C101 pad 1: Net-(C101-Pad1) -> /Clock reference/OE_A
- C205 pad 1: /Clock reference/REFIN_PRI -> /Clock reference/Input Clocks/REFIN_C
- C205 pad 2: /Clock reference/REFIN_R -> /Clock reference/Input Clocks/REFIN
- C206 pad 2: /Clock reference/REFIN_GND -> /Clock reference/Input Clocks/REFIN_GND
- C208 pad 2: /Clock reference/~CLKIN_1 -> /Clock reference/~{CLKIN_1}
- C216 pad 2: /Clock reference/CLKIN_CENTER -> /Clock reference/Input Clocks/CLKIN_CENTER
- C218 pad 1: /Clock reference/~CLKIN_1 -> /Clock reference/~{CLKIN_1}
- C227 pad 1: /Clock reference/Vctrl -> Net-(C227-Pad1)
- C234 pad 1: /Clock reference/VDD_TCXO -> /Clock reference/Input Clocks/VDD_TCXO
- C235 pad 1: /Clock reference/ERR_INP -> /Clock reference/Input Clocks/ERR_INP
- C235 pad 2: /Clock reference/DUTY_OUT_N -> /Clock reference/Input Clocks/DUTY_OUT_N
- C236 pad 1: /Clock reference/VDD_TCXO -> /Clock reference/Input Clocks/VDD_TCXO
- D105 pad 7: /Clock reference/~DF_CORR_EN -> /Clock reference/~{DF_CORR_EN}
- D201 pad 1: /Clock reference/REFIN_GND -> /Clock reference/Input Clocks/REFIN_GND
- D202 pad 1: /Clock reference/REFIN_GND -> /Clock reference/REFOUT_GND
- D202 pad 2: /Clock reference/REFIN_PRI -> /Clock reference/REFOUT_SEC
- D203 pad 1: /Clock reference/REFIN_PRI -> /Clock reference/REFOUT_SEC
- D203 pad 2: /Clock reference/REFIN_GND -> /Clock reference/REFOUT_GND
- D207 pad 1: Net-(D207-Pad1) -> /Clock reference/Input Clocks/DUTY_OUT_N
- D207 pad 2: /Clock reference/DUTY_OUT_P -> Net-(D207-Pad2)
- D208 pad 1: /Clock reference/DUTY_OUT_P -> Net-(D207-Pad2)
- D208 pad 2: Net-(D207-Pad1) -> /Clock reference/Input Clocks/DUTY_OUT_N
- FB204 pad 2: /Clock reference/VDD_TCXO -> /Clock reference/Input Clocks/VDD_TCXO
- J201 pad 1: /Clock reference/REFIN -> /Clock reference/Input Clocks/REFIN
- J201 pad 2: /Clock reference/REFIN_GND -> /Clock reference/Input Clocks/REFIN_GND
- J202 pad 1: Net-(C203-Pad1) -> Net-(J202-Pad1)
- J203 pad 1: Net-(C208-Pad1) -> Net-(J203-Pad1)
- J208 pad 1: /Clock reference/Vctrl -> Net-(C227-Pad1)
- JP202 pad 1: /Clock reference/~CLKIN_1 -> /Clock reference/~{CLKIN_1}
- JP206 pad 1: /Clock reference/~CLKIN_1 -> /Clock reference/~{CLKIN_1}
- R103 pad 1: /PLL/PLL_ON -> GND
- R103 pad 2: Net-(C101-Pad1) -> /LOS_INT
- R105 pad 1: /PLL/SCK -> GND
- R105 pad 2: Net-(C102-Pad1) -> /LOS_EXT
- R107 pad 1: /PLL/SDI -> GND
- R107 pad 2: Net-(C103-Pad1) -> /MCU/VCC_fREF
- R108 pad 1: /PLL/MUXout -> /MCU/VCC_TCXO
- R108 pad 2: Net-(C104-Pad1) -> /VCC_TCXO
- R109 pad 1: /PLL/CSB -> GND
- R109 pad 2: Net-(C105-Pad1) -> /MCU/VCC_TCXO
- R110 pad 1: /PLL/CE -> GND
- R110 pad 2: Net-(C106-Pad1) -> /MCU/VCC_PLL
- R123 pad 1: /Clock reference/~DF_CORR_EN -> /Clock reference/~{DF_CORR_EN}
- R131 pad 1: Net-(D107-Pad6) -> /MCU/VCC_fREF
- R132 pad 1: Net-(D107-Pad5) -> /MCU/VCC_PLL
- R201 pad 2: /Clock reference/REFIN_GND -> /Clock reference/Input Clocks/REFIN_GND
- R202 pad 2: Net-(C203-Pad1) -> Net-(J202-Pad1)
- R203 pad 1: /Clock reference/REFIN_R -> /Clock reference/REFOUT_SEC
- R203 pad 2: /Clock reference/REFIN -> Net-(D202-Pad3)
- R204 pad 1: /Clock reference/REFIN_GND -> /Clock reference/Input Clocks/REFIN_GND
- R204 pad 2: /Clock reference/REFIN_R -> /Clock reference/Input Clocks/REFIN
- R207 pad 2: Net-(C208-Pad1) -> Net-(J203-Pad1)
- R208 pad 1: Net-(D202-Pad3) -> /Clock reference/Input Clocks/REFIN_C
- R208 pad 2: /Clock reference/REFIN_GND -> /Clock reference/Input Clocks/REFIN_GND
- R219 pad 1: Net-(D204-Pad3) -> Net-(D202-Pad3)
- R220 pad 1: /Clock reference/CLKIN_CENTER -> /Clock reference/Input Clocks/CLKIN_CENTER
- R220 pad 2: /Clock reference/CLKIN_1 -> Net-(R217-Pad1)
- R221 pad 1: /Clock reference/~CLKIN_1 -> Net-(R218-Pad1)
- R221 pad 2: /Clock reference/CLKIN_CENTER -> /Clock reference/Input Clocks/CLKIN_CENTER
- R222 pad 1: /Clock reference/CLKIN_1 -> Net-(R217-Pad1)
- R222 pad 2: /Clock reference/DUTY_OUT_P -> /Clock reference/Input Clocks/DUTY_OUT_P
- R223 pad 1: /Clock reference/~CLKIN_1 -> Net-(R218-Pad1)
- R223 pad 2: /Clock reference/DUTY_OUT_N -> /Clock reference/Input Clocks/DUTY_OUT_N
- R224 pad 1: /Clock reference/VREF -> /Clock reference/Input Clocks/VREF
- R224 pad 2: /Clock reference/CLKIN_CENTER -> /Clock reference/Input Clocks/CLKIN_CENTER
- R225 pad 2: /Clock reference/CLKIN_CENTER -> /Clock reference/Input Clocks/CLKIN_CENTER
- R227 pad 1: /Clock reference/DUTY_OUT_N -> /Clock reference/Input Clocks/DUTY_OUT_P
- R227 pad 2: Net-(D207-Pad1) -> Net-(D207-Pad2)
- R236 pad 2: /Clock reference/Vctrl -> /Clock reference/Input Clocks/Vctrl
- R240 pad 1: /Clock reference/VDD_TCXO -> /VCC_TCXO
- R240 pad 2: /Clock reference/Vctrl -> /Clock reference/Input Clocks/Vctrl
- R241 pad 1: /Clock reference/Vctrl -> /Clock reference/Input Clocks/Vctrl
- R242 pad 1: /Clock reference/Vctrl -> /Clock reference/Input Clocks/Vctrl
- R245 pad 2: /Clock reference/ERR_INP -> /Clock reference/Input Clocks/ERR_INP
- R247 pad 1: /VCC_fREF -> /VCC_TCXO
- R249 pad 2: /Clock reference/DUTY_OUT_N -> /Clock reference/Input Clocks/DUTY_OUT_N
- R251 pad 2: /Clock reference/DUTY_OUT_P -> /Clock reference/Input Clocks/DUTY_OUT_P
- R252 pad 2: /Clock reference/~DF_CORR_EN -> /Clock reference/~{DF_CORR_EN}
- R253 pad 1: /Clock reference/VDD_TCXO -> /VCC_fREF
- R255 pad 1: /Clock reference/VDD_TCXO -> /VCC_fREF
- R306 pad 2: /PLL/SCK -> /MCU/SCK
- R309 pad 2: /PLL/SDI -> /MCU/SDI
- R311 pad 2: /PLL/MUXout -> /MCU/MUXout
- R312 pad 2: /PLL/RampDir -> /MCU/RampDir
- R313 pad 2: /PLL/CSB -> /MCU/CSB
- R314 pad 2: /PLL/RampClk -> /MCU/RampClk
- R315 pad 2: /PLL/CE -> /MCU/CE
- R325 pad 1: /PLL/PLL_ON -> /MCU/PLL_ON
- R327 pad 1: /PLL/PLL_ON -> /MCU/PLL_ON
- RV201 pad 1: /Clock reference/VDD_TCXO -> /VCC_TCXO
- T201 pad 1: /Clock reference/REFIN_PRI -> /Clock reference/Input Clocks/REFIN_PRI
- T201 pad 2: /Clock reference/REFIN_GND -> /Clock reference/Input Clocks/REFIN_GND
- T201 pad 3: Net-(C218-Pad2) -> Net-(JP502-Pad1)
- T201 pad 4: /Clock reference/CLKIN_CENTER -> /Clock reference/Input Clocks/CLKIN_CENTER
- T201 pad 5: Net-(C217-Pad2) -> Net-(JP501-Pad1)
- U201 pad 15: /Clock reference/~CLKIN_1 -> /Clock reference/~{CLKIN_1}
- U203 pad 6: /Clock reference/ERR_INP -> /Clock reference/Input Clocks/ERR_INP
- U203 pad 7: /Clock reference/DUTY_OUT_N -> /Clock reference/Input Clocks/DUTY_OUT_N
- U203 pad 8: /Clock reference/DUTY_OUT_P -> /Clock reference/Input Clocks/DUTY_OUT_P
- U204 pad 1: /Clock reference/ERR_INP -> /Clock reference/Input Clocks/DUTY_OUT_N
- U204 pad 2: /Clock reference/DUTY_OUT_N -> /Clock reference/Input Clocks/ERR_INP
- U204 pad 4: /Clock reference/~DF_CORR_EN -> /Clock reference/~{DF_CORR_EN}
- U204 pad 5: /VCC_fREF -> <NO NET>
- U301 pad 1: /PLL/CE -> /MCU/CE
- U301 pad 16: /PLL/SCK -> /MCU/SCK
- U301 pad 17: /PLL/SDI -> /MCU/SDI
- U301 pad 20: /PLL/MUXout -> /MCU/MUXout
- U301 pad 24: /PLL/CSB -> /MCU/CSB
- U301 pad 30: /PLL/RampClk -> /MCU/RampClk
- U301 pad 32: /PLL/RampDir -> /MCU/RampDir
- X201 pad 4: /Clock reference/VDD_TCXO -> /Clock reference/Input Clocks/VDD_TCXO
Routing:
- net /PLL/MUXout: track 15.9 -> 0.00 mm, vias 2 -> 0
- net /MCU/MUXout: track 0.00 -> 15.9 mm, vias 0 -> 2
- net /PLL/CSB: track 14.2 -> 0.00 mm, vias 2 -> 0
- net /MCU/CSB: track 0.00 -> 14.2 mm, vias 0 -> 2
- net /PLL/SDI: track 12.9 -> 0.00 mm
- net /MCU/SDI: track 0.00 -> 12.9 mm
- net /PLL/SCK: track 12.5 -> 0.00 mm
- net /MCU/SCK: track 0.00 -> 12.5 mm
- net /PLL/CE: track 8.49 -> 0.00 mm
- net /MCU/CE: track 0.00 -> 8.49 mm
- net /PLL/RampClk: track 6.54 -> 0.00 mm
- net /MCU/RampClk: track 0.00 -> 6.54 mm
- net /PLL/RampDir: track 5.74 -> 0.00 mm
- net /MCU/RampDir: track 0.00 -> 5.74 mm
- net Net-(J202-Pad1): track 0.00 -> 5.53 mm
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
Commit message: Synchronised PCB and schematic.
Parts:
- removed C102, C103, C104, C105, C106, C107, C108, C109, C110, C111, C112, C113, C114, C115, C116, C117, C118, C119, C120, C121: TODO, Capacitor_SMD:C_0603_1608Metric_Pad1.08x0.95mm_HandSolder
- removed C203, C208: DNP, Capacitor_SMD:C_0603_1608Metric_Pad1.08x0.95mm_HandSolder
- removed C336, C337, C339: 10n, Capacitor_SMD:C_0603_1608Metric_Pad1.08x0.95mm_HandSolder
- removed D104, D105, D107: WE-TVS-824014883, Package_DFN_QFN:UDFN-9_1.0x3.8mm_P0.5mm
- removed D204, D205, D209: BAV99, Package_TO_SOT_SMD:SOT-23
- removed D206: 1.5KE51CA, Diode_THT:D_DO-201AE_P15.24mm_Horizontal
- removed D405, D406, D407, D408: , LED_SMD:LED_0603_1608Metric_Pad1.05x0.95mm_HandSolder
- removed JP201, JP202: SolderJumper_2_Open, Jumper:SolderJumper-2_P1.3mm_Open_RoundedPad1.0x1.5mm
- removed JP503: SolderJumper_2_Bridged, Jumper:SolderJumper-2_P1.3mm_Bridged_RoundedPad1.0x1.5mm
- removed R111, R112, R113, R114, R115, R116, R117, R118, R119, R120, R121, R122, R123, R125, R126: TODO, Resistor_SMD:R_0603_1608Metric_Pad0.98x0.95mm_HandSolder
- removed R124: 3k3, Resistor_SMD:R_0603_1608Metric_Pad0.98x0.95mm_HandSolder
- removed R133, R134, R135, R136: 0R, Resistor_SMD:R_0805_2012Metric_Pad1.20x1.40mm_HandSolder
- removed R213, R214: 47, Resistor_SMD:R_0603_1608Metric_Pad0.98x0.95mm_HandSolder
- removed U402: 74HC4094, Package_SO:SO-16_3.9x9.9mm_P1.27mm
- added C420: 100n, Capacitor_SMD:C_0603_1608Metric_Pad1.08x0.95mm_HandSolder, F.Cu at (330.2, 0.00)
- added D503: SMAJ48CA, Diode_SMD_AKL:D_SMA_TVS, F.Cu at (143.3, 90.6)
- added F401: TODO, Fuse:Fuse_2920_7451Metric_Pad2.10x5.45mm_HandSolder, F.Cu at (317.8, -2.20)
- added J210: RFShield_TwoPieces, RF_Shielding:Laird_Technologies_BMI-S-205-F_38.10x25.40mm, F.Cu at (332.8, -26.9)
- added JP101: SolderJumper_2_Open, Jumper:SolderJumper-2_P1.3mm_Open_TrianglePad1.0x1.5mm, F.Cu at (371.3, -35.5)
- added JP102: SolderJumper_2_Open, Jumper:SolderJumper-2_P1.3mm_Open_TrianglePad1.0x1.5mm, F.Cu at (371.3, -31.9)
- added JP103: SolderJumper_2_Open, Jumper:SolderJumper-2_P1.3mm_Open_TrianglePad1.0x1.5mm, F.Cu at (371.3, -39.0)
- added JP104: SolderJumper_2_Open, Jumper:SolderJumper-2_P1.3mm_Open_TrianglePad1.0x1.5mm, F.Cu at (375.6, -39.0)
- added Q401: BC807, Package_TO_SOT_SMD:SOT-23, F.Cu at (330.5, -3.48)
- added Q402: BC807, Package_TO_SOT_SMD:SOT-23, F.Cu at (315.0, 7.98)
- added Q403: BC807, Package_TO_SOT_SMD:SOT-23, F.Cu at (325.6, -3.48)
- added Q404: BC807, Package_TO_SOT_SMD:SOT-23, F.Cu at (315.0, 12.4)
- added Q405: BC807, Package_TO_SOT_SMD:SOT-23, F.Cu at (319.9, 7.98)
- added Q406: BC807, Package_TO_SOT_SMD:SOT-23, F.Cu at (325.6, 0.97)
- added Q407: BC807, Package_TO_SOT_SMD:SOT-23, F.Cu at (315.0, 3.53)
- added Q408: BC807, Package_TO_SOT_SMD:SOT-23, F.Cu at (319.9, 3.53)
- added R429: 3k3, Resistor_SMD:R_0603_1608Metric_Pad0.98x0.95mm_HandSolder, F.Cu at (324.5, 4.45)
- added TP101: TestPoint_Small, TestPoint:TestPoint_Pad_D1.0mm, F.Cu at (387.2, -33.2)
- added TP102: TestPoint_Small, TestPoint:TestPoint_Pad_D1.0mm, F.Cu at (373.7, -28.6)
- added TP103: TestPoint_Small, TestPoint:TestPoint_Pad_D1.0mm, F.Cu at (375.0, -32.7)
- added TP104: TestPoint_Small, TestPoint:TestPoint_Pad_D1.0mm, F.Cu at (384.1, -36.2)
- added TP105: TestPoint_Small, TestPoint:TestPoint_Pad_D1.0mm, F.Cu at (384.1, -33.2)
- added TP106: TestPoint_Small, TestPoint:TestPoint_Pad_D1.0mm, F.Cu at (390.2, -33.2)
- added TP107: TestPoint_Small, TestPoint:TestPoint_Pad_D1.0mm, F.Cu at (378.1, -32.7)
- added TP108: TestPoint_Small, TestPoint:TestPoint_Pad_D1.0mm, F.Cu at (385.4, -39.3)
- added TP109: TestPoint_Small, TestPoint:TestPoint_Pad_D1.0mm, F.Cu at (375.0, -35.7)
- added TP110: TestPoint_Small, TestPoint:TestPoint_Pad_D1.0mm, F.Cu at (390.2, -36.2)
- added TP111: TestPoint_Small, TestPoint:TestPoint_Pad_D1.0mm, F.Cu at (381.1, -36.2)
- added TP112: TestPoint_Small, TestPoint:TestPoint_Pad_D1.0mm, F.Cu at (370.6, -28.6)
- added TP113: TestPoint_Small, TestPoint:TestPoint_Pad_D1.0mm, F.Cu at (381.1, -33.2)
- added TP114: TestPoint_Small, TestPoint:TestPoint_Pad_D1.0mm, F.Cu at (379.4, -39.3)
- added TP115: TestPoint_Small, TestPoint:TestPoint_Pad_D1.0mm, F.Cu at (388.5, -39.3)
- added TP116: TestPoint_Small, TestPoint:TestPoint_Pad_D1.0mm, F.Cu at (378.1, -35.7)
- added TP117: TestPoint_Small, TestPoint:TestPoint_Pad_D1.0mm, F.Cu at (382.4, -39.3)
- added TP118: TestPoint_Small, TestPoint:TestPoint_Pad_D1.0mm, F.Cu at (376.8, -29.6)
- added TP119: TestPoint_Small, TestPoint:TestPoint_Pad_D1.0mm, F.Cu at (385.9, -30.1)
- added TP120: TestPoint_Small, TestPoint:TestPoint_Pad_D1.0mm, F.Cu at (387.2, -36.2)
- added TP121: TestPoint_Small, TestPoint:TestPoint_Pad_D1.0mm, F.Cu at (382.9, -30.1)
- added TP122: TestPoint_Small, TestPoint:TestPoint_Pad_D1.0mm, F.Cu at (379.8, -29.6)
- added TP123: TestPoint_Small, TestPoint:TestPoint_Pad_D1.0mm, F.Cu at (391.6, -39.3)
- added TP401: TestPoint_Small, TestPoint:TestPoint_Pad_D1.0mm, F.Cu at (328.2, 4.72)
- added TP402: TestPoint_Small, TestPoint:TestPoint_Pad_D1.0mm, F.Cu at (323.8, 7.23)
- added TP403: TestPoint_Small, TestPoint:TestPoint_Pad_D1.0mm, F.Cu at (314.1, 16.2)
- added TP404: TestPoint_Small, TestPoint:TestPoint_Pad_D1.0mm, F.Cu at (318.9, 11.7)
- added TP405: TestPoint_Small, TestPoint:TestPoint_Pad_D1.0mm, F.Cu at (334.4, -4.18)
- C219, C233, C310, C326, C406, C419: footprint Capacitor_SMD:CP_Elec_6.3x7.7 -> Capacitor_SMD:CP_Elec_6.3x5.8
- C404: value 100n -> 10u; footprint Capacitor_SMD:C_0603_1608Metric_Pad1.08x0.95mm_HandSolder -> Capacitor_SMD:C_0805_2012Metric_Pad1.18x1.45mm_HandSolder
- D201: value 1.5KE51CA -> SMAJ48CA; footprint Diode_THT:D_DO-201AE_P15.24mm_Horizontal -> Diode_SMD_AKL:D_SMA_TVS
- J101: value Conn_01x02 -> POWER
- J201, J207, J304, J305, J306, J307: footprint petr_kicad:SMA_rosenberger_hybrid -> petr:SMA_rosenberger_hybrid
- J401: value Conn_01x07 -> EXPANSION; footprint Connector_PinHeader_2.54mm:PinHeader_1x07_P2.54mm_Vertical -> Connector_FFC-FPC:TE_84952-6_1x06-1MP_P1.0mm_Horizontal
- J402: value Conn_01x03 -> RS485_1
- J403: value Conn_01x03 -> RS485_2
- J404: footprint Connector_PinHeader_1.27mm:PinHeader_2x05_P1.27mm_Vertical_SMD -> petr:ArmHeader_2x05-1_P1.27mm_Vertical_SMD_pin7removed
- R401, R402, R403, R415: value 100 -> 10
- R404: value 10k -> NC
- R405: value 3k3 -> 2k
- R410, R411, R412, R413: value 2k -> 100
- R414: value 10k -> 100
- R428: value 10k -> 220
- T201, T202: footprint Transformer_SMD:Transformer_MACOM_SM-22 -> petr:Transformer_MiniCircuits_AT224-1A
- U201: footprint petr_kicad:QFN-32_EP_5x5_Pitch0.5mm_Si53301 -> petr:QFN-32_EP_5x5_Pitch0.5mm_Si53301
- U301: footprint petr_kicad:QFN-40_EP_6x6_Pitch0.5mm_LMX2572 -> petr:QFN-40_EP_6x6_Pitch0.5mm_LMX2572
- U401: value 74HC4094 -> TCA9535RTWR; footprint Package_SO:SO-16_3.9x9.9mm_P1.27mm -> Package_DFN_QFN:WQFN-24-1EP_4x4mm_P0.5mm_EP2.45x2.45mm
- U403: value efm32pg22c200f512im40-c -> EFM32PG22C200F512IM40; footprint EFM32PG22C200:efm32pg22c200f512im40-c -> petr:EFM32PG22C200F512IM40
- Y401: value 38.4 MHz -> Abracon_ABM11; footprint Crystal:Crystal_SMD_2016-4Pin_2.0x1.6mm -> petr:Crystal_SMD_Abracon_ABM3-4Pin_2.0x1.6mm
- moved X201 20.2 mm to (139.7, 63.5)
- moved J401 16.7 mm to (317.5, 63.5)
Connections:
- net Net-(D411-Pad3) renamed /MCU/RS485_A
- C229 pad 1: /VCC_fREF -> VCC_fREF
- C231 pad 1: /VCC_fREF -> VCC_fREF
- C233 pad 1: /VCC_fREF -> VCC_fREF
- C239 pad 1: /VCC_fREF -> VCC_fREF
- C402 pad 1: /MCU/VCC_MCU -> +5V
- C403 pad 1: /MCU/VCC_MCU -> /MCU/VCC_AUX
- C404 pad 2: GND -> /MCU/I2C_B
- C501 pad 1: /VCC_fREF -> VCC_fREF
- D201 pad 1: /Clock reference/Input Clocks/REFIN_GND -> GND
- D201 pad 2: GND -> /Clock reference/REFOUT_GND
- D210 pad 2: /VCC_fREF -> VCC_fREF
- D411 pad 1: Net-(D411-Pad1) -> /MCU/RS485_B
- D411 pad 4: Net-(D411-Pad4) -> unconnected-(D411-Pad4)
- D411 pad 5: /MCU/VCC_MCU -> unconnected-(D411-Pad5)
- D501 pad 2: /VCC_fREF -> VCC_fREF
- J209 pad 1: /VCC_fREF -> VCC_fREF
- J401 pad 1: /MCU/VCC_MCU -> Net-(F401-Pad2)
- J401 pad 6: Net-(D411-Pad4) -> GND
- J402 pad 2: Net-(D411-Pad1) -> GND
- J402 pad 3: GND -> /MCU/RS485_B
- J403 pad 2: Net-(D411-Pad1) -> GND
- J403 pad 3: GND -> /MCU/RS485_B
- R102 pad 2: /VCC_fREF -> VCC_fREF
- R106 pad 2: /VCC_fREF -> VCC_fREF
- R127 pad 1: /VCC_fREF -> VCC_fREF
- R129 pad 1: /VCC_fREF -> VCC_fREF
- R131 pad 2: /VCC_fREF -> VCC_fREF
- R205 pad 1: /VCC_fREF -> VCC_fREF
- R206 pad 1: /VCC_fREF -> VCC_fREF
- R209 pad 1: /VCC_fREF -> VCC_fREF
- R224 pad 1: /Clock reference/Input Clocks/VREF -> /Clock reference/VREF
- R232 pad 2: /VCC_fREF -> VCC_fREF
- R253 pad 1: /VCC_fREF -> VCC_fREF
- R255 pad 1: /VCC_fREF -> VCC_fREF
- R401 pad 1: /MCU/AUX_CLK -> /MCU/EXP_SCL
- R402 pad 1: Net-(R402-Pad1) -> /MCU/EXP_SDA
- R403 pad 1: /MCU/AUX_STR -> /MCU/~{EXP_INT}
- R404 pad 1: GND -> Net-(R404-Pad1)
- R404 pad 2: /Clock reference/CLK_SEL -> /MCU/~{EXP_INT}
- R410 pad 1: Net-(D405-Pad1) -> /MCU/VCC_MCU
- R410 pad 2: GND -> Net-(Q401-Pad2)
- R411 pad 1: Net-(D406-Pad1) -> /MCU/VCC_MCU
- R411 pad 2: GND -> Net-(Q402-Pad2)
- R412 pad 1: Net-(D407-Pad1) -> /MCU/VCC_MCU
- R412 pad 2: GND -> Net-(Q403-Pad2)
- R413 pad 1: Net-(D408-Pad1) -> /MCU/VCC_MCU
- R413 pad 2: GND -> Net-(Q404-Pad2)
- R414 pad 1: GND -> /MCU/VCC_MCU
- R414 pad 2: /MCU/AUX_OE -> Net-(Q405-Pad2)
- R415 pad 1: /MCU/AUX_OE -> /MCU/EXP_RSVD
- R418 pad 2: Net-(D411-Pad1) -> /MCU/RS485_B
- R427 pad 1: /MCU/AUX_MISO -> /MCU/VCC_MCU
- R427 pad 2: Net-(D411-Pad4) -> Net-(Q406-Pad2)
- R428 pad 1: GND -> /MCU/VCC_MCU
- R428 pad 2: /MCU/AUX_MISO -> Net-(Q408-Pad2)
- U202 pad 5: /VCC_fREF -> VCC_fREF
- U203 pad 4: /VCC_fREF -> VCC_fREF
- U204 pad 5: <NO NET> -> VCC_fREF
- U401 pad 1: /MCU/AUX_STR -> /MCU/PLL_ON
- U401 pad 10: Net-(U401-Pad10) -> /Clock reference/SFOUTB_0
- U401 pad 11: /MCU/RampDir -> /Clock reference/SFOUTB_1
- U401 pad 13: /Clock reference/OE_B -> /MCU/RampDir
- U401 pad 14: /Clock reference/~{DF_CORR_EN} -> Net-(D401-Pad2)
- U401 pad 15: /MCU/AUX_OE -> Net-(D402-Pad2)
- U401 pad 16: /MCU/VCC_MCU -> Net-(D403-Pad2)
- U401 pad 2: /MCU/AUX_D -> /Clock reference/fREF_ON
- U401 pad 3: /MCU/AUX_CLK -> /Clock reference/TCXO_ON
- U401 pad 4: /MCU/PLL_ON -> /Clock reference/CLK_SEL
- U401 pad 5: /Clock reference/fREF_ON -> /Clock reference/~{DF_CORR_EN}
- U401 pad 6: /Clock reference/TCXO_ON -> /Clock reference/OE_B
- U401 pad 7: /Clock reference/CLK_SEL -> /Clock reference/DIVA
- U401 pad 8: GND -> /Clock reference/DIVB
- U401 pad 9: unconnected-(U401-Pad9) -> GND
- U403 pad 1: /MCU/AUX_CLK -> /Clock reference/Input Clocks/DUTY_OUT_N
- U403 pad 16: /LOS_EXT -> /MCU/AUX_SDA
- U403 pad 17: /LOS_INT -> /MCU/AUX_SCL
- U403 pad 2: /MCU/AUX_D -> /MCU/VCC_PLL
- U403 pad 3: /MCU/AUX_STR -> /MCU/VCC_fREF
- U403 pad 37: /Clock reference/SFOUTB_1 -> Net-(TP405-Pad1)
- U403 pad 38: /Clock reference/SFOUTB_0 -> Net-(TP404-Pad1)
- U403 pad 39: /Clock reference/DIVB -> Net-(TP403-Pad1)
- U403 pad 4: /MCU/AUX_OE -> /MCU/EXP_SCL
- U403 pad 40: /Clock reference/DIVA -> Net-(TP402-Pad1)
- U403 pad 5: /MCU/AUX_MISO -> /MCU/EXP_SDA
- U403 pad 6: /Clock reference/Input Clocks/DUTY_OUT_N -> /MCU/~{EXP_INT}
- U403 pad 7: /MCU/VCC_PLL -> /LOS_INT
- U403 pad 8: /MCU/VCC_fREF -> /LOS_EXT
- U404 pad 7: Net-(D411-Pad1) -> /MCU/RS485_B
Routing:
- net Net-(J203-Pad1): track 0.00 -> 5.46 mm
- net Net-(C208-Pad1): track 5.46 -> 0.00 mm
- net VCC_fREF: track 0.00 -> 1.89 mm
- net /VCC_fREF: track 1.89 -> 0.00 mm

Commit message: Some minor fixes
Connections:
- C403 pad 1: /MCU/VCC_AUX -> /MCU/VCC_MCU

Commit message: Minor improvements and fixes to schematic, added high current LDO needed for high frequency PLLs.
Parts:
- C306, C307, C308, C309: value 100p -> 270p
- R428: value 220 -> 270
- R429: value 3k3 -> 2k2
Changed lines of the file:
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@@
       (effects (font (size 1 1) (thickness 0.15)))
     )
-    (fp_text value "220" (at 0 1.43) (layer "F.Fab")
+    (fp_text value "270" (at 0 1.43) (layer "F.Fab")
       (effects (font (size 1 1) (thickness 0.15)))
     )
@@
       (effects (font (size 1 1) (thickness 0.15)))
     )
-    (fp_text value "100p" (at 0 1.43) (layer "F.Fab")
+    (fp_text value "270p" (at 0 1.43) (layer "F.Fab")
       (effects (font (size 1 1) (thickness 0.15)))
     )
@@
       (effects (font (size 1 1) (thickness 0.15)))
     )
-    (fp_text value "3k3" (at 0 1.43) (layer "F.Fab")
+    (fp_text value "2k2" (at 0 1.43) (layer "F.Fab")
       (effects (font (size 1 1) (thickness 0.15)))
     )
@@
       (effects (font (size 1 1) (thickness 0.15)))
     )
-    (fp_text value "100p" (at 0 1.43) (layer "F.Fab")
+    (fp_text value "270p" (at 0 1.43) (layer "F.Fab")
       (effects (font (size 1 1) (thickness 0.15)))
     )
@@
       (effects (font (size 1 1) (thickness 0.15)))
     )
-    (fp_text value "100p" (at 0 1.43) (layer "F.Fab")
+    (fp_text value "270p" (at 0 1.43) (layer "F.Fab")
       (effects (font (size 1 1) (thickness 0.15)))
     )
@@
       (effects (font (size 1 1) (thickness 0.15)))
     )
-    (fp_text value "100p" (at 0 1.43) (layer "F.Fab")
+    (fp_text value "270p" (at 0 1.43) (layer "F.Fab")
       (effects (font (size 1 1) (thickness 0.15)))
     )
