File: PLL.kicad_sch (KiCad schematic)
At the start: 89 parts, among them J301 Vtune, J302 RFShield_TwoPieces, J303 CPout, J304 DNP, J305 DNP, J306 DNP, J307 DNP, J308 DNP, J309 RFShield_TwoPieces, U301 LMX2572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

Commit message: Fixes.
Other:
- title: Generator 0.0125 - 6.4 GHz (0.02 - 9.8 GHz) -> Generator 0.0125 - 6.4 GHz (or up to 20 GHz)
Changed lines of the file:
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@@
   (paper "A4")
   (title_block
-    (title "Generator 0.0125 - 6.4 GHz (0.02 - 9.8 GHz)")
-    (date "2021-11-13")
-    (rev "211113-001")
+    (title "Generator 0.0125 - 6.4 GHz (or up to 20 GHz)")
+    (date "2021-12-30")
+    (rev "211230-001")
     (company "Petr Polasek")
-    (comment 1 "001, 2021-11-13 09:38")
-    (comment 2 "TCXO / external input, LMX2572/LMX2592")
-    (comment 3 "Dual channel symmetric outputs")
+    (comment 1 "001, 2021-12-30 00:50")
+    (comment 2 "TCXO / external input")
+    (comment 3 "LMX2572 (6.4 GHz) / LMX2592 (9.8GHz) / LMX2594 (15 GHz) / LMX2595 (20 GHz)")
   )
   (junction (at 29.21 176.53) (diameter 1.016) (color 0 0 0 0)

Commit message: Synchronised PCB and schematic.
Parts:
- J304, J305, J306, J307: footprint petr_kicad:SMA_rosenberger_hybrid -> petr:SMA_rosenberger_hybrid
- U301: footprint petr_kicad:QFN-40_EP_6x6_Pitch0.5mm_LMX2572 -> petr:QFN-40_EP_6x6_Pitch0.5mm_LMX2572
Changed lines of the file:
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@@
     (property "Reference" "U301" (id 0) (at 67.31 158.4768 0))
     (property "Value" "LMX2572" (id 1) (at 82.55 158.2355 0))
-    (property "Footprint" "petr_kicad:QFN-40_EP_6x6_Pitch0.5mm_LMX2572" (id 2) (at 69.85 149.86 0)
+    (property "Footprint" "petr:QFN-40_EP_6x6_Pitch0.5mm_LMX2572" (id 2) (at 69.85 149.86 0)
       (effects (font (size 1.27 1.27)) hide)
     )
@@
       (effects (font (size 1.27 1.27)) (justify left))
     )
-    (property "Footprint" "petr_kicad:SMA_rosenberger_hybrid" (id 2) (at 144.78 166.37 0)
+    (property "Footprint" "petr:SMA_rosenberger_hybrid" (id 2) (at 144.78 166.37 0)
       (effects (font (size 1.27 1.27)) hide)
     )
@@
       (effects (font (size 1.27 1.27)) (justify left))
     )
-    (property "Footprint" "petr_kicad:QFN-40_EP_6x6_Pitch0.5mm_LMX2572" (id 2) (at 176.53 81.28 0)
+    (property "Footprint" "petr:QFN-40_EP_6x6_Pitch0.5mm_LMX2572" (id 2) (at 176.53 81.28 0)
       (effects (font (size 1.27 1.27)) hide)
     )
@@
       (effects (font (size 1.27 1.27)) (justify left))
     )
-    (property "Footprint" "petr_kicad:SMA_rosenberger_hybrid" (id 2) (at 167.64 182.88 0)
+    (property "Footprint" "petr:SMA_rosenberger_hybrid" (id 2) (at 167.64 182.88 0)
       (effects (font (size 1.27 1.27)) hide)
     )
@@
       (effects (font (size 1.27 1.27)) (justify left))
     )
-    (property "Footprint" "petr_kicad:SMA_rosenberger_hybrid" (id 2) (at 167.64 166.37 0)
+    (property "Footprint" "petr:SMA_rosenberger_hybrid" (id 2) (at 167.64 166.37 0)
       (effects (font (size 1.27 1.27)) hide)
     )
@@
       (effects (font (size 1.27 1.27)) (justify left))
     )
-    (property "Footprint" "petr_kicad:QFN-40_EP_6x6_Pitch0.5mm_LMX2572" (id 2) (at 129.54 80.01 0)
+    (property "Footprint" "petr:QFN-40_EP_6x6_Pitch0.5mm_LMX2572" (id 2) (at 129.54 80.01 0)
       (effects (font (size 1.27 1.27)) hide)
     )
@@
       (effects (font (size 1.27 1.27)) (justify left))
     )
-    (property "Footprint" "petr_kicad:QFN-40_EP_6x6_Pitch0.5mm_LMX2572" (id 2) (at 255.27 80.01 0)
+    (property "Footprint" "petr:QFN-40_EP_6x6_Pitch0.5mm_LMX2572" (id 2) (at 255.27 80.01 0)
       (effects (font (size 1.27 1.27)) hide)
     )
@@
       (effects (font (size 1.27 1.27)) (justify right))
     )
-    (property "Footprint" "petr_kicad:QFN-40_EP_6x6_Pitch0.5mm_LMX2572" (id 2) (at 219.71 82.55 0)
+    (property "Footprint" "petr:QFN-40_EP_6x6_Pitch0.5mm_LMX2572" (id 2) (at 219.71 82.55 0)
       (effects (font (size 1.27 1.27)) hide)
     )
@@
       (effects (font (size 1.27 1.27)) (justify left))
     )
-    (property "Footprint" "petr_kicad:SMA_rosenberger_hybrid" (id 2) (at 144.78 182.88 0)
+    (property "Footprint" "petr:SMA_rosenberger_hybrid" (id 2) (at 144.78 182.88 0)
       (effects (font (size 1.27 1.27)) hide)
     )
@@
       (effects (font (size 1.27 1.27)) (justify left))
     )
-    (property "Footprint" "petr_kicad:QFN-40_EP_6x6_Pitch0.5mm_LMX2572" (id 2) (at 83.82 26.67 0)
-      (effects (font (size 1.27 1.27)) hide)
-    )
+    (property "Footprint" "petr:QFN-40_EP_6x6_Pitch0.5mm_LMX2572" (id 2) (at 83.82 26.67 0)
+      (effects (font (size 1.27 1.27)) hide)
+    )

Commit message: Minor improvements and fixes to schematic, added high current LDO needed for high frequency PLLs.
Parts:
- added U303: AP2112K-3.3, Package_TO_SOT_SMD:SOT-23-5, symbol Regulator_Linear:AP2112K-3.3
- C306, C307, C308, C309: value 100p -> 270p
- U302: value XC6204B33 -> XC6204F33; symbol petr:XC6204B33 -> petr:XC6204F33
Connections:
- net +5V: now also U303.1 (VIN)
- net GND: now also U303.2 (GND)
- net VCC_PLL: now also U303.5 (VOUT)
- net PLL_CE: now reaches C318.1, R327.2, U302.3 (CE)
- net PLL_CE: now also U303.3 (EN)
Other:
- note added: "Replacement LDO used for higher frequency PLLs which consume >300 mA."
- moved on the sheet: C318, R325, R327
